File: Fiber_Optics/Fiber_Audio_Link_TX_RX_MM/Fiber_Audio_Link_TX_RX_MM.kicad_sch (KiCad schematic)
At the start: 43 parts, among them J1 AudioJack4, J2 Conn_01x02, J3 Conn_01x10, J4 Conn_01x02, Q1 2N2222, Q2 Q_Photo_NPN, SW1 SW_SPDT, SW2 SW_SPDT, U1 LM358P, U2 LM386

Commit message: update fiber audio link project.
Parts:
- removed J2: Conn_01x02, Connector_PinHeader_2.54mm:PinHeader_1x02_P2.54mm_Vertical, symbol Connector_Generic:Conn_01x02
- added J2: Conn_01x06, Connector_PinHeader_2.54mm:PinHeader_1x06_P2.54mm_Vertical, symbol Connector_Generic:Conn_01x06
Connections:
- net +5V: now also J2.1 (Pin_1)
- net GND: now also J2.2 (Pin_2)
- net at R3.2, RV3.2: no longer RV3.3
Other:
- moved on the sheet: C2, C3
